File: PCB/Proyecto de prueba.kicad_sch (KiCad schematic)
At the start: 8 parts, among them J1 Conn_01x02

Commit message: "footprints added"
Parts:
- added LA, LL, RA, RL: Conn_01x01, MountingHole:MountingHole_5mm, symbol Connector_Generic:Conn_01x01
Connections:
- net GND: now also RA.1 (Pin_1), RL.1 (Pin_1)
- net LA: no longer names the net of R4.2, R5.1
- net LA: now also LA.1 (Pin_1)
- net LL: no longer names the net of R3.1, R4.1
- net LL: now also LL.1 (Pin_1)
