File: electronica/kicad/Proyecto de prueba.kicad_sch (KiCad schematic)
At the start: 24 parts, among them M1 TP4056_modulo, M2 MT3608, SW1 SPST, U1 ESP32-S3-DEVKITC-1-N16R8V

Commit message: Se elimino el diodo. Se empezo el PCB
Parts:
- removed D2: 1N5819, Diode_THT:D_DO-41_SOD81_P10.16mm_Horizontal, symbol Diode:1N5819
- added C5: 100u, Capacitor_THT:CP_Radial_D6.3mm_P2.50mm, symbol Device:C
Connections:
- net 5V0: now also C4.2, M2.VOUT_P (VOUT+), C5.1; no longer C3.2, C4.1
- net GND: now also C3.2, C4.1, M1.6 (OUT-), C5.2; no longer C3.1, C4.2, M1.4 (OUT-)
- net at BT1.1 (Pin_1): now also M1.4 (B+); no longer M1.5 (B+)
- net at BT1.2 (Pin_2): now also M1.5 (B-); no longer M1.6 (B-)
- net at M2.VIN_P (VIN+), SW1.1 (A): now also C3.1
Other:
- moved on the sheet: BT1

Commit message: PCB_organized
Parts:
- removed J_BNC1: BNC, symbol Connector_Generic:Conn_01x02
- removed U1: ESP32-S3-DEVKITC-1-N16R8V, ESP32-S3-DEVKITC-1-N16R8V:XCVR_ESP32-S3-DEVKITC-1-N16R8V, symbol ESP32-S3-DEVKITC-1-N16R8V:ESP32-S3-DEVKITC-1-N16R8V
- added TP1: TP1, TestPoint:TestPoint_THTPad_D2.0mm_Drill1.0mm, symbol Connector_Generic:Conn_01x01
- added U1: ESP32-CAM, MyFootprints:ESP32-CAM, symbol ESP32-CAM:ESP32-CAM
- R4: value 330k -> 220K
Connections:
- net 5V0: now also U1.5V
- net GND: now also U1.GND2
- net PWM: now also U1.IO14
- net at R7.2: now also U1.IO4
- net at C2.1, R3.2, R4.1: now also TP1.1 (Pin_1)
- no-connect marks 38 -> 14
Other:
- moved on the sheet: D3, R7

Commit message: PCB TERMINADO
Parts:
- removed J_LA1: LA, TestPoint:TestPoint_THTPad_D2.0mm_Drill1.0mm, symbol Connector_Generic:Conn_01x01
- added C4: 100n, Capacitor_THT:C_Disc_D5.0mm_W2.5mm_P2.50mm, symbol Device:C
- added C5: 10n, Capacitor_THT:C_Disc_D5.0mm_W2.5mm_P2.50mm, symbol Device:C
- added J_LL1: LL, TestPoint:TestPoint_THTPad_D2.0mm_Drill1.0mm, symbol Connector_Generic:Conn_01x01
- added R10, R12: 200, Resistor_THT:R_Axial_DIN0207_L6.3mm_D2.5mm_P10.16mm_Horizontal, symbol Device:R
- added R11: 22K, Resistor_THT:R_Axial_DIN0207_L6.3mm_D2.5mm_P10.16mm_Horizontal, symbol Device:R
- added R3: 1k, Resistor_THT:R_Axial_DIN0207_L6.3mm_D2.5mm_P10.16mm_Horizontal, symbol Device:R
- added R4: 10k, Resistor_THT:R_Axial_DIN0207_L6.3mm_D2.5mm_P10.16mm_Horizontal, symbol Device:R
- added TP1: TP1, TestPoint:TestPoint_THTPad_D2.0mm_Drill1.0mm, symbol Connector_Generic:Conn_01x01
- added TP3: TP3, TestPoint:TestPoint_THTPad_D2.0mm_Drill1.0mm, symbol Connector_Generic:Conn_01x01
- J_LA1: renamed from J_LL1; value LL -> LA
- R5: value 100 -> 220K
- R6: value 100 -> 200
- TP2: renamed from TP1; value TP1 -> TP2
- renumbered C4 to C1, C5 to C2, C1 to C6, C2 to C7, D3 to D1, D1 to D2, M2 to M1, M1 to M2, R7 to R1, R1 to R2, R2 to R7, R3 to R8, R4 to R9
Connections:
- net GND: now also R6.1, U1.GND, U1.GND1, C4.2, C5.2, R10.1; no longer J_RA1.1 (Pin_1), R6.2
- net at R1.2: now also U1.IO12; no longer U1.IO4
- net PWM3: now reaches U1.IO13
- net PWM3: now also R11.1
- net PWM2: now reaches U1.IO15
- net PWM2: now also R7.1
- net at R5.2: now also J_RA1.1 (Pin_1), R6.2; no longer R6.1
- net at J_LA1.1 (Pin_1), R9.2: now also R10.2, R12.2; no longer R5.1
- net PWM renamed PWM1
- net PWM1: now also R3.1; no longer R7.1
- new net: C5.1, R4.2, R5.1, TP1.1 (Pin_1)
- new net: J_LL1.1 (Pin_1), R11.2, R12.1, TP3.1 (Pin_1)
- new net: C4.1, R3.2, R4.1
- no-connect marks 14 -> 10
Other:
- moved on the sheet: C3, C6, C7, D1, D2, J_LA1, R1, R2, R7, R8, R9, TP2

Commit message: Firmware_1_Electrode y 3D listo
Connections:
- net GND: no longer U1.GND1
- no-connect marks 10 -> 11
Changed lines of the file:
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@@
+	)
+	(no_connect
+		(at 190.5 44.45)
 	)
 	(no_connect
@@
 					(unit 1)
 				)
-			)
-		)
-	)
-	(symbol
-		(lib_id "power:GND")
-		(at 190.5 44.45 270)
-		(unit 1)
-		(body_style 1)
-		(exclude_from_sim no)
-		(in_bom yes)
-		(on_board yes)
-		(in_pos_files yes)
-		(dnp no)
-		(property "Reference" "#PWR05"
-			(at 184.15 44.45 0)
-			(hide yes)
-			(show_name no)
-			(do_not_autoplace no)
-			(effects
-				(font
-					(size 1.27 1.27)
-				)
-			)
-		)
-		(property "Value" "GND"
-			(at 185.928 44.704 90)
-			(show_name no)
-			(do_not_autoplace no)
-			(effects
-				(font
-					(size 1.27 1.27)
-				)
-				(justify right)
-			)
-		)
-		(property "Footprint" ""
-			(at 190.5 44.45 0)
-			(hide yes)
-			(show_name no)
-			(do_not_autoplace no)
-			(effects
-				(font
-					(size 1.27 1.27)
-				)
-			)
-		)
-		(property "Datasheet" ""
-			(at 190.5 44.45 0)
-			(hide yes)
-			(show_name no)
-			(do_not_autoplace no)
-			(effects
-				(font
-					(size 1.27 1.27)
-				)
-			)
-		)
-		(property "Description" "Power symbol creates a global label with name \"GND\" , ground"
-			(at 190.5 44.45 0)
-			(hide yes)
-			(show_name no)
-			(do_not_autoplace no)
-			(effects
-				(font
-					(size 1.27 1.27)
-				)
-			)
-		)
-		(pin "1"
-		)
-		(instances
-			(project "Proyecto de prueba"
-				(path "/a97c120f-b434-430d-8622-c04d8223901b"
-					(reference "#PWR05")
-					(unit 1)
-				)
