File: electronica/kicad/Proyecto de prueba.kicad_pcb (KiCad board)
At the start: 2 copper layers, 80 x 130 mm, 23 parts, among them M1 TP4056_modulo, M2 MT3608, SW1 SPST, U1 ESP32-S3-DEVKITC-1-N16R8V

Commit message: PCB_organized
Parts:
- removed D2: 1N5819, Diode_THT:D_DO-41_SOD81_P10.16mm_Horizontal
- added C5: 100u, Capacitor_THT:CP_Radial_D6.3mm_P2.50mm, F.Cu at (159.0, 139.0)
- added TP1: TP1, TestPoint:TestPoint_THTPad_D2.0mm_Drill1.0mm, F.Cu at (109.5, 59.0)
- R4: value 330k -> 220K
- U1: value ESP32-S3-DEVKITC-1-N16R8V -> ESP32-CAM; footprint ESP32-S3-DEVKITC-1-N16R8V:XCVR_ESP32-S3-DEVKITC-1-N16R8V -> MyFootprints:ESP32-CAM
- moved SW1 96.3 mm to (107.5, 146.0), turned to 90 degrees
- moved M1 62.7 mm to (117.7, 163.1), turned to 90 degrees
- moved M2 48.5 mm to (158.5, 154.5), turned to 180 degrees
- moved C1 48.2 mm to (119.8, 88.5)
- moved J_RA1 45.2 mm to (161.5, 68.0)
- moved C2 38.1 mm to (122.0, 67.2), turned to -90 degrees
- moved R1 37.5 mm to (181.0, 51.9), turned to -90 degrees
- moved R7 32.9 mm to (175.0, 62.1), turned to 90 degrees
- moved C3 31.1 mm to (106.5, 128.5), turned to -90 degrees
- moved J_RL1 28.4 mm to (176.0, 68.0)
- moved R4 28.0 mm to (115.9, 55.0)
- moved BT1 27.9 mm to (127.0, 130.5), turned to 180 degrees
- moved R2 27.6 mm to (114.0, 89.6), turned to 90 degrees
- moved R6 27.4 mm to (150.9, 55.0)
- moved J_LL1 26.9 mm to (130.5, 68.0)
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Connections:
- M2 pad VOUT_P: Net-(D2-A) -> /5V0
- R7 pad 2: Net-(U1-GPIO5) -> Net-(R7-Pad2)
Other:
- board size 80 x 130 mm -> 90 x 130 mm

Commit message: PCB TERMINADO
Parts:
- removed the D1 at (170.0, 46.0)
- removed the J_LA1 at (147.5, 68.0)
- added C6: 100n, Capacitor_THT:C_Disc_D5.0mm_W2.5mm_P2.50mm, F.Cu at (141.5, 69.2)
- added C7: 10n, Capacitor_THT:C_Disc_D5.0mm_W2.5mm_P2.50mm, F.Cu at (147.5, 60.5)
- added D2: VERDE_ON, LED_THT:LED_D5.0mm, F.Cu at (181.5, 47.0)
- added J_LL1: LL, TestPoint:TestPoint_THTPad_D2.0mm_Drill1.0mm, F.Cu at (165.0, 54.5)
- added R10: 200, Resistor_THT:R_Axial_DIN0207_L6.3mm_D2.5mm_P10.16mm_Horizontal, F.Cu at (157.0, 60.4)
- added R11: 22K, Resistor_THT:R_Axial_DIN0207_L6.3mm_D2.5mm_P10.16mm_Horizontal, F.Cu at (147.4, 78.0)
- added R12: 200, Resistor_THT:R_Axial_DIN0207_L6.3mm_D2.5mm_P10.16mm_Horizontal, F.Cu at (171.0, 54.9)
- added R8: 10k, Resistor_THT:R_Axial_DIN0207_L6.3mm_D2.5mm_P10.16mm_Horizontal, F.Cu at (147.5, 74.6)
- added R9: 220K, Resistor_THT:R_Axial_DIN0207_L6.3mm_D2.5mm_P10.16mm_Horizontal, F.Cu at (152.5, 64.5)
- added TP2: TP2, TestPoint:TestPoint_THTPad_D2.0mm_Drill1.0mm, F.Cu at (155.0, 49.5)
- C2: value 10n -> 100u; footprint Capacitor_THT:C_Disc_D5.0mm_W2.5mm_P2.50mm -> Capacitor_THT:CP_Radial_D6.3mm_P2.50mm
- C5: value 100u -> 10n; footprint Capacitor_THT:CP_Radial_D6.3mm_P2.50mm -> Capacitor_THT:C_Disc_D5.0mm_W2.5mm_P2.50mm
- J_LA1: renamed from J_LL1; value LL -> LA
- M1: value TP4056_modulo -> MT3608; footprint TP4056_modulo:TP4056_modulo -> MT3608_DC:MT3608_DC
- M2: value MT3608 -> TP4056_modulo; footprint MT3608_DC:MT3608_DC -> TP4056_modulo:TP4056_modulo
- R2: value 1k -> 330
- R3: value 10k -> 1k
- R4: value 220K -> 10k
- R5: value 100 -> 220K
- R6: value 100 -> 200
- R7: value 330 -> 1k
- moved C5 88.5 mm to (112.8, 63.5), turned to 180 degrees
- moved C3 73.5 mm to (178.5, 113.5), turned to 90 degrees
- moved R2 73.0 mm to (182.0, 63.1)
- moved SW1 72.8 mm to (178.5, 129.8), turned to -90 degrees
- moved M1 67.4 mm to (161.9, 112.2), turned to -90 degrees
- moved C4 63.8 mm to (112.8, 76.5)
- moved C2 61.5 mm to (176.3, 96.0), turned to 0 degrees
- moved C1 60.9 mm to (179.2, 101.5), turned to 180 degrees
- moved J_RL1 52.8 mm to (125.0, 54.5)
- moved R7 43.4 mm to (134.5, 77.6)
- moved R1 38.1 mm to (157.6, 82.0), turned to 180 degrees
- moved J_RA1 37.0 mm to (125.0, 74.0)
- moved J_LA1 35.0 mm to (165.0, 74.0)
- moved TP1 27.2 mm to (135.0, 49.5)
- moved BT1 27.2 mm to (150.0, 145.0), turned to 90 degrees
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- renumbered D3 to D1
Connections:
- C1 pad 1: Net-(C1-Pad1) -> GND
- C1 pad 2: GND -> /5V0
- C2 pad 1: Net-(TP1-Pin_1) -> /5V0
- C3 pad 1: GND -> Net-(M1-VIN+)
- C3 pad 2: /5V0 -> GND
- C4 pad 1: /5V0 -> Net-(C4-Pad1)
- C5 pad 1: /5V0 -> Net-(TP1-Pin_1)
- D1 pad 1: Net-(D3-K) -> Net-(D1-K)
- J_LA1 pad 1: Net-(J_LL1-Pin_1) -> Net-(J_LA1-Pin_1)
- J_RA1 pad 1: GND -> Net-(J_RA1-Pin_1)
- R1 pad 1: /5V0 -> Net-(D1-K)
- R1 pad 2: Net-(D1-K) -> Net-(R1-Pad2)
- R2 pad 1: /PWM -> /5V0
- R2 pad 2: Net-(C1-Pad1) -> Net-(D2-K)
- R3 pad 1: Net-(C1-Pad1) -> /PWM1
- R3 pad 2: Net-(TP1-Pin_1) -> Net-(C4-Pad1)
- R4 pad 1: Net-(TP1-Pin_1) -> Net-(C4-Pad1)
- R4 pad 2: Net-(J_LL1-Pin_1) -> Net-(TP1-Pin_1)
- R5 pad 1: Net-(J_LL1-Pin_1) -> Net-(TP1-Pin_1)
- R5 pad 2: Net-(J_LA1-Pin_1) -> Net-(J_RA1-Pin_1)
- R6 pad 1: Net-(J_LA1-Pin_1) -> GND
- R6 pad 2: GND -> Net-(J_RA1-Pin_1)
- R7 pad 1: Net-(D3-K) -> /PWM2
- R7 pad 2: Net-(R7-Pad2) -> Net-(C6-Pad1)
- SW1 pad 1: Net-(M2-VIN+) -> Net-(M1-VIN+)
- SW1 pad 2: Net-(M1-OUT+) -> Net-(M2-OUT+)
- U1 pad GND: unconnected-(U1-PadGND) -> GND
- U1 pad GND1: unconnected-(U1-PadGND1) -> GND
- U1 pad IO12: unconnected-(U1-PadIO12) -> Net-(R1-Pad2)
- U1 pad IO13: unconnected-(U1-PadIO13) -> /PWM3
- U1 pad IO14: /PWM -> /PWM1
- U1 pad IO15: unconnected-(U1-PadIO15) -> /PWM2
- U1 pad IO4: Net-(R7-Pad2) -> unconnected-(U1-PadIO4)
Routing:
- net GND: track 0.00 -> 411.3 mm
- net /5V0: track 0.00 -> 104.3 mm
- net Net-(D1-K): track 0.00 -> 55.3 mm
- net Net-(J_LL1-Pin_1): track 0.00 -> 48.9 mm
- net Net-(M1-VIN+): track 0.00 -> 45.3 mm
- net Net-(M2-OUT+): track 0.00 -> 39.6 mm
- net Net-(TP1-Pin_1): track 0.00 -> 38.8 mm
- net Net-(J_LA1-Pin_1): track 0.00 -> 27.6 mm
- net /PWM3: track 0.00 -> 26.4 mm
- net Net-(TP2-Pin_1): track 0.00 -> 23.6 mm
- net Net-(R1-Pad2): track 0.00 -> 21.4 mm
- net /PWM2: track 0.00 -> 18.0 mm
- net Net-(C6-Pad1): track 0.00 -> 16.0 mm
- net Net-(J_RA1-Pin_1): track 0.00 -> 15.4 mm
- net Net-(BT1-Pin_1): track 0.00 -> 11.9 mm
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
Commit message: Firmware_1_Electrode y 3D listo
Parts:
- added TP3: TP3, TestPoint:TestPoint_THTPad_D2.0mm_Drill1.0mm, F.Cu at (155.0, 49.5)
- moved TP2 10.0 mm to (145.0, 49.5)
- moved R10 5.08 mm to (151.9, 60.5), turned to 0 degrees
- moved U1 0.85 mm to (117.5, 103.6)
Connections:
- U1 pad GND1: GND -> unconnected-(U1-PadGND1)
Routing:
- net Net-(J_LL1-Pin_1): track 48.9 -> 61.0 mm
- net Net-(J_LA1-Pin_1): track 27.6 -> 35.0 mm
- net Net-(D2-K): track 0.00 -> 6.13 mm
- net Net-(TP2-Pin_1): track 23.6 -> 21.5 mm
- net GND: track 411.3 -> 412.4 mm
- net /5V0: track 104.3 -> 103.8 mm
Other:
- board text added: "+"
- board text added: "-"
- board text added: "ESP32 CAM"
- board text added: "GND"
- board text added: "LiPo"
- board text added: "MT3608"
- board text added: "SPST"
- board text added: "TP4056"
- board text added: "VIN_IN"
- board text added: "VIN_OUT"
